Commit message: fix xacro

File: limo_vehicle_description/urdf/vehicle.xacro (robot description, xacro)
@@ -6,5 +6,5 @@
   <link name="base_link">
     <visual>
-      <origin xyz="${vehicle_info['/**']['ros__parameters']['wheel_base']/2.0} 0 0" rpy="${pi/2.0} 0 ${pi}"/>
+      <origin xyz="${vehicle_info['/**']['ros__parameters']['wheel_base']/2.0} 0 0" rpy="0 0 ${pi/2.0}"/>
       <geometry>
         <mesh filename="package://limo_vehicle_description/mesh/limo_base.dae" scale="1 1 1"/>
